File: LED Board/LED Board 2.kicad_sch (KiCad schematic)
At the start: 10 parts, among them J1 Connector, U1 TLV62569DDC

Commit message: Add files via upload
Parts:
- R1: value 400k -> 200k
- R2: value 100k -> 50k
Changed lines of the file:
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@@
 			)
 		)
-		(property "Value" "100k"
+		(property "Value" "50k"
 			(at 157.48 104.1399 0)
 			(effects
@@
 			)
 		)
-		(property "Value" "400k"
+		(property "Value" "200k"
 			(at 157.48 96.5199 0)
 			(effects
